File: board/board.sch (KiCad schematic (older format))
At the start: 80 parts, among them IC1 LVC245A, IC2 LVC245A, J1 Conn_01x11_Male, J10 Conn_01x01_Male, J2 AudioJack4_Ground, J3 Conn_01x01_Male, J4 Conn_01x01_Male, J5 Conn_01x01_Male, J6 Conn_01x01_Male, J7 Conn_01x01_Male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

Commit message: Ongoing design
Squeezing all necessary electronics onto a 3.3mm x 5.1mm board
Parts:
- removed C26, C27: 100nF, Capacitor_SMD:C_0603_1608Metric_Pad1.05x0.95mm_HandSolder, symbol Device:C_Small
Connections:
- net labels added: PB2, PR2, Y2
- wire segments 434 -> 426
Changed lines of the file:
@@
 NoConn ~ 8950 6200
-$Comp
-L Device:C_Small C26
-U 1 1 59EA3E26
-P 1200 5600
-F 0 "C26" H 1210 5670 50  0000 L CNN
-F 1 "100nF" V 1100 5500 50  0000 L CNN
-F 2 "Capacitor_SMD:C_0603_1608Metric_Pad1.05x0.95mm_HandSolder" H 1200 5600 50  0001 C CNN
-F 3 "" H 1200 5600 50  0000 C CNN
-	1    1200 5600
-	0    1    1    0
-$EndComp
-$Comp
-L Device:C_Small C27
-U 1 1 59EA3E2C
-P 1200 5900
-F 0 "C27" H 1210 5970 50  0000 L CNN
-F 1 "100nF" V 1100 5800 50  0000 L CNN
-F 2 "Capacitor_SMD:C_0603_1608Metric_Pad1.05x0.95mm_HandSolder" H 1200 5900 50  0001 C CNN
-F 3 "" H 1200 5900 50  0000 C CNN
-	1    1200 5900
-	0    1    1    0
-$EndComp
 $Comp
 L components:LFSPXO024957 OSC1
@@
 Connection ~ 10550 5150
 Connection ~ 10550 5350
-Connection ~ 10550 5550
 Wire Wire Line
 	10450 5550 10550 5550
@@
 	10550 5750 10450 5750
 Wire Wire Line
-	11400 6750 11400 5450
+	11400 6750 11400 5650
 Wire Wire Line
 	9700 4950 10250 4950
@@
 	9350 6150 10250 6150
 Wire Wire Line
-	1350 5600 1300 5600
-Wire Wire Line
-	1050 5600 1100 5600
-Wire Wire Line
-	1350 5900 1300 5900
-Wire Wire Line
-	1050 5900 1100 5900
-Connection ~ 1350 5300
-Connection ~ 1350 5600
-Connection ~ 1050 5300
-Connection ~ 1050 5600
-Wire Wire Line
 	13450 6050 13450 6200
 Wire Wire Line
 	13150 5400 13100 5400
 Wire Wire Line
-	13100 5400 13100 5550
-Wire Wire Line
-	13100 5550 12850 5550
-Wire Wire Line
 	10550 6550 10450 6550
-Wire Wire Line
-	10550 5550 10550 5750
 Wire Wire Line
 	2800 9100 2950 9100
@@
 	1300 6800 1350 6800
 Wire Wire Line
-	11400 5450 11900 5450
-Wire Wire Line
-	11700 5650 11900 5650
-Wire Wire Line
-	11700 5150 11700 5650
-Wire Wire Line
 	13150 5850 13000 5850
 Wire Wire Line
-	13000 5850 13000 5450
-Wire Wire Line
-	13000 5450 12850 5450
-Wire Wire Line
-	12850 5650 12900 5650
-Wire Wire Line
-	12900 5650 12900 4950
+	13000 5850 13000 5650
 Wire Wire Line
 	12900 4950 13150 4950
@@
 	10550 5350 10700 5350
 Wire Wire Line
-	10550 5550 11900 5550
-Wire Wire Line
 	10550 5750 10550 5950
 Wire Wire Line
@@
 Wire Wire Line
 	12250 1950 12250 2050
-Wire Wire Line
-	1350 5300 1350 5600
-Wire Wire Line
-	1350 5600 1350 5900
-Wire Wire Line
-	1050 5300 1050 5600
-Wire Wire Line
-	1050 5600 1050 5900
 Wire Wire Line
 	2950 9100 3300 9100
@@
 L Connector:Conn_01x01_Male J10
 U 1 1 5FC22E6A
+P 7850 9950
+F 0 "J10" V 8003 9863 50  0000 R CNN
+F 1 "Conn_01x01_Male" V 7912 9863 50  0000 R CNN
+F 2 "Connector_PinHeader_2.54mm:PinHeader_1x01_P2.54mm_Vertical" H 7850 9950 50  0001 C CNN
+F 3 "~" H 7850 9950 50  0001 C CNN
+	1    7850 9950
+	0    -1   -1   0
+$EndComp
+$Comp
+L Connector:Conn_01x01_Male J3
+U 1 1 5FC23046
 P 7950 9700
-F 0 "J10" V 8103 9613 50  0000 R CNN
+F 0 "J3" V 8103 9613 50  0000 R CNN
 F 1 "Conn_01x01_Male" V 8012 9613 50  0000 R CNN
 F 2 "Connector_PinHeader_2.54mm:PinHeader_1x01_P2.54mm_Vertical" H 7950 9700 50  0001 C CNN
 F 3 "~" H 7950 9700 50  0001 C CNN
 	1    7950 9700
-	0    -1   -1   0
-$EndComp
-$Comp
-L Connector:Conn_01x01_Male J3
-U 1 1 5FC23046
-P 7850 9950
-F 0 "J3" V 8003 9863 50  0000 R CNN
-F 1 "Conn_01x01_Male" V 7912 9863 50  0000 R CNN
-F 2 "Connector_PinHeader_2.54mm:PinHeader_1x01_P2.54mm_Vertical" H 7850 9950 50  0001 C CNN
-F 3 "~" H 7850 9950 50  0001 C CNN
-	1    7850 9950
 	0    -1   -1   0
 $EndComp
@@
 Wire Wire Line
 	3700 7700 4250 7700
+Text Label 12950 4950 0    60   ~ 0
+PR2
+Text Label 13050 5850 0    60   ~ 0
+Y2
+Text Label 13100 5400 1    60   ~ 0
+PB2
+Wire Wire Line
+	13100 5400 13100 5550
+Wire Wire Line
+	12850 5550 13100 5550
+Connection ~ 10550 5550
+Wire Wire Line
+	11700 5150 11700 5450
+Wire Wire Line
+	10550 5550 10550 5750
+Wire Wire Line
+	11700 5450 11900 5450
+Wire Wire Line
+	11400 5650 11900 5650
+Wire Wire Line
+	10550 5550 11900 5550
+Wire Wire Line
+	12900 4950 12900 5450
+Wire Wire Line
+	12900 5450 12850 5450
+Wire Wire Line
+	12850 5650 13000 5650
 $EndSCHEMATC

Commit message: Layout complete (version 1)
Parts:
- removed J1: Conn_01x11_Male, Connector_PinHeader_2.54mm:PinHeader_1x11_P2.54mm_Vertical, symbol Connector:Conn_01x11_Male
- added J1: Conn_01x06_Male, Connector_PinHeader_2.54mm:PinHeader_1x06_P2.54mm_Vertical, symbol Connector:Conn_01x06_Male
- added J11: Conn_01x05_Male, Connector_PinHeader_2.54mm:PinHeader_1x05_P2.54mm_Vertical, symbol Connector:Conn_01x05_Male
Changed lines of the file:
@@
-$EndComp
-$Comp
-L Connector:Conn_01x11_Male J1
-U 1 1 5E65371C
-P 6600 800
-F 0 "J1" V 6435 776 50  0000 C CNN
-F 1 "Conn_01x11_Male" V 6526 776 50  0000 C CNN
-F 2 "Connector_PinHeader_2.54mm:PinHeader_1x11_P2.54mm_Vertical" H 6600 800 50  0001 C CNN
-F 3 "~" H 6600 800 50  0001 C CNN
-	1    6600 800
-	0    1    1    0
 $EndComp
 $Comp
@@
 Wire Wire Line
 	12850 5650 13000 5650
+$Comp
+L Connector:Conn_01x05_Male J11
+U 1 1 5E618FCE
+P 6900 800
+F 0 "J11" V 6700 750 50  0000 L CNN
+F 1 "Conn_01x05_Male" V 6800 550 50  0000 L CNN
+F 2 "Connector_PinHeader_2.54mm:PinHeader_1x05_P2.54mm_Vertical" H 6900 800 50  0001 C CNN
+F 3 "~" H 6900 800 50  0001 C CNN
+	1    6900 800
+	0    1    1    0
+$EndComp
+$Comp
+L Connector:Conn_01x06_Male J1
+U 1 1 5E619200
+P 6400 800
+F 0 "J1" V 6200 750 50  0000 L CNN
+F 1 "Conn_01x06_Male" V 6300 350 50  0000 L CNN
+F 2 "Connector_PinHeader_2.54mm:PinHeader_1x06_P2.54mm_Vertical" H 6400 800 50  0001 C CNN
+F 3 "~" H 6400 800 50  0001 C CNN
+	1    6400 800
+	0    1    1    0
+$EndComp
 $EndSCHEMATC

Commit message: Redesign mode jumpers. Minor fixes in silk screen.
Parts:
- removed J10, J3, J4: Conn_01x01_Male, Connector_PinHeader_2.54mm:PinHeader_1x01_P2.54mm_Vertical, symbol Connector:Conn_01x01_Male
- added J10, J3: Conn_01x02, Connector_PinHeader_2.54mm:PinHeader_2x01_P2.54mm_Vertical, symbol Connector_Generic:Conn_01x02
Connections:
- net labels added: RGBMODE
- net labels removed: SCANLINES
- wire segments 426 -> 431
Changed lines of the file:
@@
 	14000 1950 14150 1950
-$Comp
-L Connector:Conn_01x01_Male J4
-U 1 1 5F9AA036
-P 900 10300
-F 0 "J4" H 1006 10478 50  0000 C CNN
-F 1 "Conn_01x01_Male" H 1006 10387 50  0000 C CNN
-F 2 "Connector_PinHeader_2.54mm:PinHeader_1x01_P2.54mm_Vertical" H 900 10300 50  0001 C CNN
-F 3 "~" H 900 10300 50  0001 C CNN
-	1    900  10300
-	1    0    0    -1
-$EndComp
 $Comp
 L Connector:Conn_01x01_Male J5
@@
 $EndComp
 Wire Wire Line
-	1100 10300 1400 10300
-Wire Wire Line
 	1450 10550 1400 10550
 Wire Wire Line
@@
 Wire Wire Line
 	1400 10300 1400 10550
-Connection ~ 1400 10300
 Wire Wire Line
 	1400 10300 1450 10300
@@
 Wire Wire Line
 	13350 5850 14000 5850
-$Comp
-L Connector:Conn_01x01_Male J10
-U 1 1 5FC22E6A
-P 7850 9950
-F 0 "J10" V 8003 9863 50  0000 R CNN
-F 1 "Conn_01x01_Male" V 7912 9863 50  0000 R CNN
-F 2 "Connector_PinHeader_2.54mm:PinHeader_1x01_P2.54mm_Vertical" H 7850 9950 50  0001 C CNN
-F 3 "~" H 7850 9950 50  0001 C CNN
-	1    7850 9950
-	0    -1   -1   0
-$EndComp
-$Comp
-L Connector:Conn_01x01_Male J3
-U 1 1 5FC23046
-P 7950 9700
-F 0 "J3" V 8103 9613 50  0000 R CNN
-F 1 "Conn_01x01_Male" V 8012 9613 50  0000 R CNN
-F 2 "Connector_PinHeader_2.54mm:PinHeader_1x01_P2.54mm_Vertical" H 7950 9700 50  0001 C CNN
-F 3 "~" H 7950 9700 50  0001 C CNN
-	1    7950 9700
-	0    -1   -1   0
-$EndComp
 Text Label 7850 9100 3    60   ~ 0
 LINEDOUBLE
 Text Label 7950 9450 1    60   ~ 0
-SCANLINES
-Wire Wire Line
-	7850 8600 7850 9750
-Wire Wire Line
-	7950 8600 7950 9500
+RGBMODE
 $Comp
 L power:PWR_FLAG #FLG0101
@@
 	0    1    1    0
 $EndComp
+$Comp
+L Connector_Generic:Conn_01x02 J10
+U 1 1 5EC27787
+P 8400 10350
+F 0 "J10" V 8273 10430 50  0000 L CNN
+F 1 "Conn_01x02" V 8364 10430 50  0000 L CNN
+F 2 "Connector_PinHeader_2.54mm:PinHeader_2x01_P2.54mm_Vertical" H 8400 10350 50  0001 C CNN
+F 3 "~" H 8400 10350 50  0001 C CNN
+	1    8400 10350
+	0    1    1    0
+$EndComp
+$Comp
+L Connector_Generic:Conn_01x02 J3
+U 1 1 5EC278B2
+P 8400 9850
+F 0 "J3" V 8273 9930 50  0000 L CNN
+F 1 "Conn_01x02" V 8364 9930 50  0000 L CNN
+F 2 "Connector_PinHeader_2.54mm:PinHeader_2x01_P2.54mm_Vertical" H 8400 9850 50  0001 C CNN
+F 3 "~" H 8400 9850 50  0001 C CNN
+	1    8400 9850
+	0    1    1    0
+$EndComp
+Wire Wire Line
+	7850 10050 8300 10050
+Wire Wire Line
+	8300 10050 8300 10150
+Wire Wire Line
+	7850 8600 7850 10050
+$Comp
+L power:GND #PWR0106
+U 1 1 5ECB44FC
+P 8400 10050
+F 0 "#PWR0106" H 8400 9800 50  0001 C CNN
+F 1 "GND" V 8405 9922 50  0000 R CNN
+F 2 "" H 8400 10050 50  0001 C CNN
+F 3 "" H 8400 10050 50  0001 C CNN
+	1    8400 10050
+	0    -1   -1   0
+$EndComp
+$Comp
+L power:GND #PWR0107
+U 1 1 5ECB46A9
+P 8400 9550
+F 0 "#PWR0107" H 8400 9300 50  0001 C CNN
+F 1 "GND" V 8405 9422 50  0000 R CNN
+F 2 "" H 8400 9550 50  0001 C CNN
+F 3 "" H 8400 9550 50  0001 C CNN
+	1    8400 9550
+	0    -1   -1   0
+$EndComp
+Wire Wire Line
+	8400 9650 8400 9550
+Wire Wire Line
+	8400 10150 8400 10050
+Wire Wire Line
+	7950 9550 8300 9550
+Wire Wire Line
+	8300 9550 8300 9650
+Wire Wire Line
+	7950 8600 7950 9550
 $EndSCHEMATC
